Commit message: ball detected

File: install/akabot_description/share/akabot_description/urdf/akabot_tf_camera.xacro (robot description, xacro)
@@ -3,5 +3,6 @@
   <xacro:property name="pole_height" value="0.8" />
   <xacro:property name="pole_radius" value="0.015" />
-  <xacro:property name="pole_x" value="0.3" /> <xacro:property name="pole_y" value="0.4" /> <link name="camera_pole_link">
+  <xacro:property name="pole_x" value="0.3" /> <xacro:property name="pole_y" value="0.4" />
+  <link name="camera_pole_link">
     <visual>
       <origin xyz="0 0 ${pole_height/2}" rpy="0 0 0"/>
