Commit message: solve the left_claw_joint error

File: install/akabot_description/share/akabot_description/urdf/akabot.ros2_control.xacro (robot description, xacro)
@@ -1,17 +1,16 @@
 <?xml version="1.0"?>
 <robot xmlns:xacro="http://www.ros.org/wiki/xacro">
-  <!-- Properties -->
   <xacro:property name="initial_positions_file" value="$(find akabot_description)/config/initial_positions.yaml"/>
   <xacro:property name="initial_positions" value="${xacro.load_yaml(initial_positions_file)['initial_positions']}"/>
-  <!-- ros2_control macro -->
   <xacro:macro name="akabot_ros2_control" params="name plugin_name">
     <ros2_control name="${name}" type="system">
       <hardware>
-        <plugin>gz_ros2_control/GazeboSimSystem</plugin>
+        <plugin>${plugin_name}</plugin>
       </hardware>
       <joint name="top_plate_joint">
-        <command_interface name="position"/>
+        <command_interface name="position">
           <param name="min">1.56</param>
           <param name="max">4.68</param>
+        </command_interface>
         <state_interface name="position">
           <param name="initial_value">${initial_positions['top_plate_joint']}</param>
@@ -20,7 +19,8 @@
       </joint>
       <joint name="lower_arm_joint">
-        <command_interface name="position"/>
+        <command_interface name="position">
           <param name="min">0.0</param>
           <param name="max">3.12</param>
+        </command_interface>
         <state_interface name="position">
           <param name="initial_value">${initial_positions['lower_arm_joint']}</param>
@@ -29,7 +29,8 @@
       </joint>
       <joint name="upper_arm_joint">
-        <command_interface name="position"/>
+        <command_interface name="position">
           <param name="min">-1.7</param>
           <param name="max">1.7</param>
+        </command_interface>
         <state_interface name="position">
           <param name="initial_value">${initial_positions['upper_arm_joint']}</param>
@@ -38,7 +39,8 @@
       </joint>
       <joint name="wrist_joint">
-        <command_interface name="position"/>
+        <command_interface name="position">
           <param name="min">-1.7</param>
           <param name="max">1.7</param>
+        </command_interface>
         <state_interface name="position">
           <param name="initial_value">${initial_positions['wrist_joint']}</param>
@@ -47,7 +49,8 @@
       </joint>
       <joint name="claw_base_joint">
-        <command_interface name="position"/>
+        <command_interface name="position">
           <param name="min">-3.17</param>
           <param name="max">0.0</param>
+        </command_interface>
         <state_interface name="position">
           <param name="initial_value">${initial_positions['claw_base_joint']}</param>
@@ -56,7 +59,8 @@
       </joint>
       <joint name="right_claw_joint">
-        <command_interface name="position"/>
+        <command_interface name="position">
           <param name="min">-0.5</param>
           <param name="max">0.0</param>
+        </command_interface>
         <state_interface name="position">
           <param name="initial_value">${initial_positions['right_claw_joint']}</param>
@@ -65,6 +69,4 @@
       </joint>
       <joint name="left_claw_joint">
-        <param name="mimic">right_claw_joint</param>
-        <param name="multiplier">-1</param>
         <command_interface name="position"/>
           <param name="min">0.0</param>

File: install/akabot_description/share/akabot_description/urdf/akabot_core.xacro (robot description, xacro)
@@ -14,5 +14,5 @@
     <parent link="base_link"/>
     <child link="base_plate"/>
-    <origin xyz="0 0 0"/>
+    <origin xyz="0.1 0.05 0"/>
   </joint>
   <!-- Base plate -->
@@ -40,5 +40,5 @@
     <parent link="base_plate"/>
     <child link="top_plate"/>
-    <origin rpy="0 0 1.5" xyz="0 0 0.048"/>
+    <origin rpy="0 0 1.5" xyz="0.0 0 0.048"/>
     <axis xyz="0 0 1" />
     <limit effort="1000.0" lower="1.56" upper="4.68" velocity="1.0" />
@@ -217,5 +217,4 @@
     <axis xyz="0 0 1" />
     <limit effort="1000.0" lower="0.0" upper="0.5" velocity="1.0" />
-    <mimic joint="right_claw_joint" multiplier="-1" offset="0" />
   </joint>
 </robot>

File: install/akabot_description/share/akabot_description/urdf/akabot_gz.urdf.xacro (robot description, xacro)
@@ -4,7 +4,7 @@
     <xacro:include filename="$(find akabot_description)/urdf/akabot.ros2_control.xacro"/>
     <!-- <xacro:include filename="$(find akabot_description)/urdf/depth_camera.xacro"/> -->
-    <xacro:akabot_ros2_control name="IgnitionSystem" plugin_name="ign_ros2_control/IgnitionSystem"/>
+    <xacro:akabot_ros2_control name="GazeboSimSystem" plugin_name="gz_ros2_control/GazeboSimSystem"/>
     <gazebo>
-      <plugin filename="libign_ros2_control-system.so" name="ign_ros2_control::IgnitionROS2ControlPlugin">
+      <plugin filename="libgz_ros2_control-system.so" name="gz_ros2_control::GazeboSimROS2ControlPlugin">
         <parameters>$(find akabot_bringup)/config/ros2_controllers.yaml</parameters>
       </plugin>

File: src/akabot_description/urdf/akabot_core.xacro (robot description, xacro)
@@ -14,5 +14,5 @@
     <parent link="base_link"/>
     <child link="base_plate"/>
-    <origin xyz="0 0 0"/>
+    <origin xyz="0.1 0.05 0"/>
   </joint>
   <!-- Base plate -->
@@ -40,5 +40,5 @@
     <parent link="base_plate"/>
     <child link="top_plate"/>
-    <origin rpy="0 0 1.5" xyz="0 0 0.048"/>
+    <origin rpy="0 0 1.5" xyz="0.0 0 0.15"/>
     <axis xyz="0 0 1" />
     <limit effort="1000.0" lower="1.56" upper="4.68" velocity="1.0" />
@@ -217,5 +217,4 @@
     <axis xyz="0 0 1" />
     <limit effort="1000.0" lower="0.0" upper="0.5" velocity="1.0" />
-    <mimic joint="right_claw_joint" multiplier="-1" offset="0" />
   </joint>
 </robot>
