Commit message: Fix mimic joint error by removing explicit mimic joint from ros2_control

File: src/akabot_description/urdf/akabot.ros2_control.xacro (robot description, xacro)
@@ -64,15 +64,7 @@
         <state_interface name="velocity"/>
       </joint>
-      <joint name="left_claw_joint">
-        <param name="mimic">right_claw_joint</param>
-        <param name="multiplier">-1</param>
-        <command_interface name="position"/>
-          <param name="min">0.0</param>
-          <param name="max">0.5</param>
-        <state_interface name="position">
-          <param name="initial_value">${initial_positions['left_claw_joint']}</param>
-        </state_interface>
-        <state_interface name="velocity"/>
-      </joint>
+      <!-- FIXED: Removed explicit mimic joint from ros2_control -->
+      <!-- The left_claw_joint is a mimic joint in URDF and will be automatically handled -->
+      <!-- Do NOT add a separate ros2_control entry for mimic joints -->
     </ros2_control>
   </xacro:macro>
